File: Hardware/PCB_Rack/PCB_Rack.kicad_pcb (KiCad board)
At the start: 2 copper layers, 433.9 x 44.5 mm, 73 parts, among them J1 Conn_01x03, J2 Conn_01x03, J3 Conn_01x03, J4 Conn_01x03, J5 Conn_01x03, J6 Conn_01x03, J7 Conn_01x03, Q1 IRLML6244, Q10 IRLML6244, Q11 IRLML6244, Q12 IRLML6244, Q2 IRLML6244, Q3 IRLML6244, Q4 IRLML6244, Q5 IRLML6244, Q6 IRLML6244, Q7 IRLML6244, Q8 IRLML6244, Q9 IRLML6244, SW1 SW_SPST, SW2 SW_SPST, U3 PCF8575DBR

Commit message: finalisation PCB Rack
Parts:
- added C12: 4u7, Capacitor_SMD:C_0603_1608Metric_Pad1.08x0.95mm_HandSolder, F.Cu at (155.0, 187.7)
- added H7: MountingHole_Pad, MountingHole:MountingHole_2.2mm_M2_DIN965_Pad_TopBottom, F.Cu at (402.0, 189.1)
- H3, H4: footprint MountingHole:MountingHole_3.2mm_M3_DIN965_Pad_TopBottom -> MountingHole:MountingHole_2.2mm_M2_DIN965_Pad_TopBottom
- moved J5 57.9 mm to (369.9, 188.0)
- moved J6 57.9 mm to (419.9, 188.0)
- moved J7 57.9 mm to (468.0, 188.1)
- moved J4 57.9 mm to (321.4, 188.0)
- moved J3 57.8 mm to (268.8, 188.0)
- moved J2 57.7 mm to (217.0, 188.0)
- moved R5 52.9 mm to (169.5, 179.3), turned to -90 degrees
- moved D1 51.4 mm to (154.7, 185.0), turned to 0 degrees
- moved C3 49.9 mm to (149.8, 184.7)
- moved H4 49.6 mm to (303.2, 189.1)
- moved R2 49.6 mm to (142.3, 175.8)
- moved R1 49.5 mm to (146.8, 175.8)
- moved C4 49.4 mm to (151.1, 175.8)
- moved SW2 49.4 mm to (144.2, 170.2)
- moved H3 49.3 mm to (231.3, 189.0)
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Connections:
- net Net-(J2-Pin_1) renamed /Relais1/LINE_Sw
- net Net-(J3-Pin_1) renamed /Relais2/LINE_Sw
- net Net-(J4-Pin_1) renamed /Relais3/LINE_Sw
- net Net-(J5-Pin_1) renamed /Relais4/LINE_Sw
- net Net-(J6-Pin_1) renamed /Relais5/LINE_Sw
- net Net-(J7-Pin_1) renamed /Relais6/LINE_Sw
Routing:
- net /INA6_2: track 0.00 -> 339.1 mm, vias 0 -> 1
- net /INA6_1: track 0.00 -> 318.2 mm, vias 0 -> 1
- net /INA5_2: track 0.00 -> 285.0 mm, vias 0 -> 1
- net /INA5_1: track 0.00 -> 262.4 mm, vias 0 -> 1
- net /INA4_2: track 0.00 -> 221.7 mm, vias 0 -> 1
- net /INA4_1: track 0.00 -> 204.6 mm, vias 0 -> 1
- net /INA3_2: track 0.00 -> 167.1 mm, vias 0 -> 1
- net /INA3_1: track 0.00 -> 147.9 mm, vias 0 -> 1
- net /INA2_2: track 0.00 -> 116.7 mm, vias 0 -> 1
- net /INA2_1: track 0.00 -> 97.5 mm, vias 0 -> 1
- net +5V: track 0.00 -> 70.1 mm, vias 0 -> 2
- net /INA1_2: track 0.00 -> 63.9 mm, vias 0 -> 1
- net Net-(D5-DOUT): track 0.00 -> 50.2 mm
- net Net-(D7-DOUT): track 0.00 -> 48.3 mm
- net Net-(D3-DOUT): track 0.00 -> 47.8 mm
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- added copper zone on F.Cu, net +5V
- added copper zone on F.Cu, net /Phase
- added copper zone on F.Cu, net /Relais1/LINE_Sw
- added copper zone on F.Cu, net /Relais2/LINE_Sw
- added copper zone on F.Cu, net /Relais3/LINE_Sw
- added copper zone on F.Cu, net /Relais4/LINE_Sw
- added copper zone on F.Cu, net /Relais5/LINE_Sw
- added copper zone on F.Cu, net /Relais6/LINE_Sw
- added copper zone on F.Cu, net Earth
- added copper zone on B.Cu, net GND
- added copper zone on F.Cu, net GND
- added copper zone on F.Cu, net LINE
- added copper zone on B.Cu, net NEUT
Other:
- board size 433.9 x 44.5 mm -> 420.8 x 44.5 mm

Commit message: finalisation PCB routagev2
Parts:
- added G***: LOGO, img:Dessin_CoventGarden, B.Cu at (132.7, 198.6)
- C1, C12: moved to B.Cu
- U1: footprint ESP32_C3_SuperMini:C3_SuperMini -> ESP32_C3_SuperMini:SuperMini SMT
- moved U1 15.9 mm to (164.4, 176.3)
- moved R6 6.72 mm to (175.0, 179.2), turned to 180 degrees
- moved R5 5.87 mm to (175.0, 177.2), turned to 180 degrees
- moved C1 4.99 mm to (156.6, 188.3), turned to 0 degrees
- moved C12 4.51 mm to (152.6, 183.9), turned to 90 degrees
- moved C5 0.60 mm to (127.2, 174.9)
- moved U3 0.57 mm to (133.0, 172.5)
- moved R11 0.26 mm to (283.4, 177.3)
- moved R18 0.10 mm to (451.3, 177.2)
Routing:
- net +5V: track 70.1 -> 47.9 mm, vias 2 -> 10
- net /INA5_1: track 262.4 -> 270.0 mm
- net /INA5_2: track 285.0 -> 290.5 mm
- net /INA6_2: track 339.1 -> 344.5 mm
- net SCL: track 46.6 -> 52.0 mm, vias 0 -> 1
- net /INA6_1: track 318.2 -> 323.4 mm
- net /INA4_1: track 204.6 -> 202.1 mm
- net /INA3_2: track 167.1 -> 169.4 mm
- net /INA3_1: track 147.9 -> 150.2 mm
- net /INA1_2: track 63.9 -> 66.1 mm
- net /INA4_2: track 221.7 -> 219.7 mm
- net Px: track 24.8 -> 23.1 mm, vias 0 -> 1
- net /INA2_2: track 116.7 -> 118.2 mm
- net SDA: track 47.4 -> 48.7 mm, vias 0 -> 1
- net /INA1_1: track 46.9 -> 48.1 mm
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- added copper zone on B.Cu, net +5V
Other:
- board text added: "Alim_5V"
- board text added: "By Capodagli Janus"
- board text added: "COVENT"
- board text added: "GARDEN"
- board text added: "STUDIOS"
