File: Hardware/PCB_Rack/PCB_Rack.kicad_pcb (KiCad board)
At the start: 2 copper layers, 420.8 x 44.5 mm, 76 parts, among them J1 Conn_01x03, J2 Conn_01x03, J3 Conn_01x03, J4 Conn_01x03, J5 Conn_01x03, J6 Conn_01x03, J7 Conn_01x03, Q1 IRLML6244, Q10 IRLML6244, Q11 IRLML6244, Q12 IRLML6244, Q2 IRLML6244, Q3 IRLML6244, Q4 IRLML6244, Q5 IRLML6244, Q6 IRLML6244, Q7 IRLML6244, Q8 IRLML6244, Q9 IRLML6244, SW1 SW_SPST, SW2 SW_SPST, U3 PCF8575DBR

Commit message: maj pcb
Routing:
- net /INA6_1: track 323.4 -> 324.4 mm
- net Net-(SW2-A): track 8.58 -> 9.28 mm
- net GND: vias 597 -> 601

Commit message: update LOGO
Parts:
- added G***: LOGO, img:Logo_Covent, B.Cu at (118.3, 204.5)
- Q1, Q10, Q11, Q12, Q2, Q3, Q4, Q5, Q6, Q7, Q8, Q9: value IRLML6244 -> SQ2310ES-T1_BE3
- moved G*** 15.0 mm to (118.8, 193.0)
Other:
- board text removed: "COVENT"
- board text removed: "GARDEN"
- board text removed: "STUDIOS"

Commit message: 49.3
Parts:
- removed U4, U5, U6, U7, U8, U9: ~, Relais_Bistable_SPDT:SPDT_bistable
- added G***: LOGO, img:ARDUINO, B.Cu at (117.3, 184.6)
- added U10: ~, Relais_Bistable_SPDT:SPDY_Bistable_1fromC, B.Cu at (191.8, 189.6)
- added U11: ~, Relais_Bistable_SPDT:SPDY_Bistable_1fromC, B.Cu at (242.0, 189.6)
- added U12: ~, Relais_Bistable_SPDT:SPDY_Bistable_1fromC, B.Cu at (292.0, 189.6)
- added U13: ~, Relais_Bistable_SPDT:SPDY_Bistable_1fromC, B.Cu at (343.6, 189.6)
- added U14: ~, Relais_Bistable_SPDT:SPDY_Bistable_1fromC, B.Cu at (391.6, 189.5)
- added U15: ~, Relais_Bistable_SPDT:SPDY_Bistable_1fromC, B.Cu at (441.6, 189.5)
- moved G*** 27.8 mm to (145.0, 202.3)
- moved C10 3.29 mm to (396.4, 173.5)
- moved C8 3.20 mm to (297.5, 173.6)
Routing:
- net Net-(Q11-D): track 6.61 -> 8.96 mm
- net Net-(Q12-D): track 4.85 -> 7.07 mm
- net Net-(Q1-D): track 6.52 -> 8.68 mm
- net Net-(Q6-D): track 5.18 -> 7.31 mm
- net Net-(Q9-D): track 7.04 -> 9.17 mm
- net Net-(Q10-D): track 5.30 -> 7.43 mm
- net Net-(Q4-D): track 5.32 -> 7.37 mm
- net Net-(Q3-D): track 7.22 -> 9.27 mm
- net Net-(Q8-D): track 3.97 -> 6.01 mm
- net Net-(Q7-D): track 6.99 -> 9.04 mm
- net Net-(Q2-D): track 4.51 -> 6.31 mm
- net Net-(Q5-D): track 6.77 -> 8.44 mm
- net GND: vias 601 -> 608

Commit message: Correction footprint connecteurs
Parts:
- H1, H2, H5, H6: footprint MountingHole:MountingHole_3.2mm_M3_DIN965_Pad_TopBottom -> MountingHole:MountingHole_2.2mm_M2_DIN965_Pad_TopBottom
- J2, J3, J4, J5, J6, J7: footprint Conn_Alim:Conn_Secteur -> Conn_Alim:Conn_Secteur_femelle
- moved J5 6.75 mm to (363.2, 188.0)
- moved J7 6.05 mm to (462.0, 188.3)
- moved J6 6.05 mm to (413.9, 188.0)
- moved J4 5.91 mm to (315.5, 188.0)
- moved J2 5.50 mm to (211.5, 188.2)
- moved J3 5.19 mm to (263.6, 188.0)
- moved H5 1.41 mm to (478.0, 206.2)
- moved H6 1.41 mm to (478.0, 169.8)
- moved R18 0.38 mm to (450.9, 177.2)
- moved Q12 0.34 mm to (450.7, 180.0)
Routing:
- net Net-(D4-DOUT): track 44.6 -> 45.2 mm
- net GND: vias 608 -> 630

Commit message: maj pcb
Parts:
- removed the G*** at (117.3, 184.6)
- moved G*** 28.9 mm to (118.0, 192.0)

Commit message: ajout des pulldown sur les transistors
Parts:
- added R19: 10k, Resistor_SMD:R_0603_1608Metric_Pad0.98x0.95mm_HandSolder, B.Cu at (179.4, 178.3)
- added R20: 10k, Resistor_SMD:R_0603_1608Metric_Pad0.98x0.95mm_HandSolder, B.Cu at (229.4, 180.1)
- added R21: 10k, Resistor_SMD:R_0603_1608Metric_Pad0.98x0.95mm_HandSolder, B.Cu at (280.8, 177.4)
- added R22: 10k, Resistor_SMD:R_0603_1608Metric_Pad0.98x0.95mm_HandSolder, B.Cu at (334.6, 175.2)
- added R23: 10k, Resistor_SMD:R_0603_1608Metric_Pad0.98x0.95mm_HandSolder, B.Cu at (384.0, 174.4)
- added R24: 10k, Resistor_SMD:R_0603_1608Metric_Pad0.98x0.95mm_HandSolder, B.Cu at (434.1, 174.4)
- added R25: 10k, Resistor_SMD:R_0603_1608Metric_Pad0.98x0.95mm_HandSolder, B.Cu at (200.5, 175.2)
- added R26: 10k, Resistor_SMD:R_0603_1608Metric_Pad0.98x0.95mm_HandSolder, B.Cu at (251.9, 175.3)
- added R27: 10k, Resistor_SMD:R_0603_1608Metric_Pad0.98x0.95mm_HandSolder, B.Cu at (305.5, 180.0)
- added R28: 10k, Resistor_SMD:R_0603_1608Metric_Pad0.98x0.95mm_HandSolder, B.Cu at (352.4, 175.0)
- added R29: 10k, Resistor_SMD:R_0603_1608Metric_Pad0.98x0.95mm_HandSolder, B.Cu at (404.2, 180.5)
- added R30: 10k, Resistor_SMD:R_0603_1608Metric_Pad0.98x0.95mm_HandSolder, B.Cu at (452.2, 174.2)
- moved R8 0.46 mm to (200.5, 177.5)
- moved C9 0.37 mm to (341.0, 174.2)
Routing:
- net Net-(Q12-G): track 2.15 -> 8.12 mm
- net Net-(Q4-G): track 2.16 -> 7.88 mm
- net Net-(Q7-G): track 2.23 -> 7.88 mm
- net Net-(Q11-G): track 2.06 -> 7.55 mm
- net Net-(Q8-G): track 1.95 -> 7.10 mm
- net Net-(Q9-G): track 2.16 -> 6.79 mm
- net Net-(Q3-G): track 2.15 -> 5.82 mm
- net Net-(Q5-G): track 2.04 -> 5.61 mm
- net Net-(Q1-G): track 2.23 -> 5.72 mm
- net Net-(Q6-G): track 2.16 -> 5.03 mm
- net Net-(Q10-G): track 2.12 -> 4.76 mm
- net /INA1_1: track 48.0 -> 50.2 mm
- net /INA3_1: track 150.3 -> 152.1 mm
- net Net-(Q2-G): track 2.16 -> 4.00 mm
- net /INA1_2: track 66.1 -> 67.3 mm
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
Commit message: ajout des pinheaders en plus
Parts:
- added J10: Conn_01x04, Connector_PinHeader_2.54mm:PinHeader_1x04_P2.54mm_Vertical, F.Cu at (167.5, 183.7)
- added J8: Conn_01x04, Connector_PinHeader_2.54mm:PinHeader_1x04_P2.54mm_Vertical, F.Cu at (165.0, 183.7)
- added J9: Conn_01x04, Connector_PinHeader_2.54mm:PinHeader_1x04_P2.54mm_Vertical, F.Cu at (162.4, 183.7)
- moved R5 12.3 mm to (163.2, 173.7)
- moved R6 10.8 mm to (164.9, 175.4)
- moved U14 1.67 mm to (391.6, 191.2)
- moved U15 1.67 mm to (441.6, 191.2)
- moved U11 1.64 mm to (242.0, 191.2)
- moved U13 1.62 mm to (343.6, 191.2)
- moved U12 1.60 mm to (292.0, 191.2)
- moved U10 1.58 mm to (191.8, 191.2)
Connections:
- U1 pad 10: unconnected-(U1-GPIO6-Pad10) -> /GPIO6
- U1 pad 11: unconnected-(U1-GPIO7-Pad11) -> /GPIO7
- U1 pad 12: SDA -> /GPIO8
- U1 pad 13: SCL -> SDA
- U1 pad 4: unconnected-(U1-GPIO3-Pad4) -> SCL
- U1 pad 5: unconnected-(U1-GPIO4-Pad5) -> Px
- U1 pad 6: unconnected-(U1-3.3V-Pad6) -> +3.3V
- U1 pad 9: Px -> /GPIO5
Routing:
- net /GPIO8: track 0.00 -> 11.6 mm
- net +3.3V: track 0.00 -> 11.6 mm
- net /GPIO6: track 0.00 -> 11.0 mm
- net /GPIO7: track 0.00 -> 8.02 mm
- net /GPIO5: track 0.00 -> 7.73 mm
- net Px: track 23.1 -> 29.5 mm
- net SCL: track 52.0 -> 45.6 mm
- net +5V: track 47.9 -> 52.3 mm
- net Net-(Q11-D): track 8.96 -> 6.45 mm
- net SDA: track 48.7 -> 46.5 mm
- net Net-(Q10-D): track 7.43 -> 5.35 mm
- net Net-(Q12-D): track 7.12 -> 5.05 mm
- net Net-(Q2-D): track 6.31 -> 4.27 mm
- net Net-(Q7-D): track 9.04 -> 7.13 mm
- net Net-(Q4-D): track 7.37 -> 5.48 mm
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- added copper zone on B.Cu, net +3.3V
Other:
- board text added: "3.3V"
- board text added: "5V"
- board text added: "Gnd"
- board text added: "IO"
- board text added: "Vcc"

Commit message: correction orientation des connecteurs sur secteur
Parts:
- added G***: LOGO, img:Logo_Covent, F.Cu at (217.8, 205.8)
- added G***: LOGO, img:dessin_musique, B.Cu at (137.0, 198.7)
- D2: footprint LED_SMD:LED_0603_1608Metric_Pad1.05x0.95mm_HandSolder -> img:LED_0603_avec_dessin
- moved G*** 32.8 mm to (148.8, 203.2)
- moved J7 9.16 mm to (471.1, 187.9), turned to -90 degrees
- moved J6 8.41 mm to (422.3, 187.9), turned to -90 degrees
- moved J5 8.13 mm to (371.3, 187.9), turned to -90 degrees
- moved J2 8.01 mm to (219.5, 187.9), turned to -90 degrees
- moved J4 7.60 mm to (323.1, 187.9), turned to -90 degrees
- moved J3 7.18 mm to (270.8, 187.9), turned to -90 degrees
- moved D2 6.47 mm to (112.6, 174.5), turned to 0 degrees
- moved R3 1.87 mm to (118.3, 177.1), turned to -90 degrees
Routing:
- net Net-(D2-A): track 2.04 -> 9.81 mm
- net GND: vias 797 -> 821
Other:
- board text removed: "Alim_5V"
