File: Hardware/PCB_Rack/PCB_Rack.kicad_pcb (KiCad board)
At the start: 2 copper layers, 420.8 x 44.5 mm, 94 parts, among them J1 Conn_01x03, J10 Conn_01x04, J2 Conn_01x03, J3 Conn_01x03, J4 Conn_01x03, J5 Conn_01x03, J6 Conn_01x03, J7 Conn_01x03, J8 Conn_01x04, J9 Conn_01x04, Q1 SQ2310ES-T1_BE3, Q10 SQ2310ES-T1_BE3, Q11 SQ2310ES-T1_BE3, Q12 SQ2310ES-T1_BE3, Q2 SQ2310ES-T1_BE3, Q3 SQ2310ES-T1_BE3, Q4 SQ2310ES-T1_BE3, Q5 SQ2310ES-T1_BE3, Q6 SQ2310ES-T1_BE3, Q7 SQ2310ES-T1_BE3, Q8 SQ2310ES-T1_BE3, Q9 SQ2310ES-T1_BE3, SW1 SW_SPST, SW2 SW_SPST, U3 PCF8575DBR

Commit message: correction des pull-up sur SDA/SCL, finalisation du code esp32 Google_Calendar pour que la reconnexion (sur google device)se fasse automatiquement après reboot
Parts:
- added C13: 22u, Capacitor_SMD:C_0201_0603Metric_Pad0.64x0.40mm_HandSolder, F.Cu at (173.5, 190.8)
- added C14: 10u, Capacitor_SMD:C_0201_0603Metric_Pad0.64x0.40mm_HandSolder, F.Cu at (178.5, 188.0)
- added U4: AZ1117-3.3, Package_TO_SOT_SMD:SOT-223-3_TabPin2, F.Cu at (174.2, 185.8)
- moved U3 40.2 mm to (173.1, 175.7)
- moved C5 39.0 mm to (165.8, 179.8), turned to 0 degrees
- moved D2 15.9 mm to (128.5, 175.0)
- moved R3 15.9 mm to (134.1, 177.6)
- moved R5 3.63 mm to (165.8, 176.2), turned to -90 degrees
- moved R6 2.86 mm to (163.2, 177.8), turned to -90 degrees
Connections:
- C5 pad 2: +5V -> +3.3V
- J10 pad 1: /GPIO8 -> /GPIO4
- R5 pad 1: +5V -> +3.3V
- R6 pad 1: +5V -> +3.3V
- U1 pad 12: /GPIO8 -> Px
- U1 pad 5: Px -> /GPIO4
- U1 pad 6: +3.3V -> unconnected-(U1-3.3V-Pad6)
- U3 pad 24: +5V -> +3.3V
Routing:
- net /INA1_1: track 50.2 -> 5.76 mm
- net /INA4_1: track 203.0 -> 158.9 mm
- net /INA3_2: track 170.4 -> 126.3 mm
- net /INA6_2: track 344.6 -> 300.6 mm
- net /INA4_2: track 220.7 -> 176.7 mm
- net /INA6_1: track 324.5 -> 280.6 mm
- net /INA5_2: track 291.0 -> 247.3 mm
- net /INA5_1: track 270.1 -> 226.5 mm
- net /INA3_1: track 152.1 -> 108.8 mm
- net /INA2_2: track 119.3 -> 76.3 mm
- net /INA2_1: track 99.6 -> 57.1 mm
- net /INA1_2: track 67.3 -> 25.2 mm
- net +5V: track 52.3 -> 15.9 mm, vias 10 -> 9
- net SDA: track 46.5 -> 13.2 mm
- net SCL: track 45.6 -> 15.8 mm
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- added copper zone on F.Cu, net +3.3V

Commit message: maj README, ajout 3D boitier afficheur, 3D repetition, firmware Rack
Parts:
- C3: value 100u -> 220u
Changed lines of the file:
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@@
 			)
 		)
-		(property "Value" "100u"
+		(property "Value" "220u"
 			(at 0 -1.5 90)
 			(unlocked yes)
@@
 			(keep_text_aligned yes)
 		)
-		(gr_text "420,75"
+		(gr_text "420.75"
 			(at 271.625 156.98 0)
 			(layer "Dwgs.User")
@@
 			(keep_text_aligned yes)
 		)
-		(gr_text "44,45"
+		(gr_text "44.45"
 			(at 48.81 187.965 90)
 			(layer "Dwgs.User")
