File: Hardware/PCB_Repetition/XLR.kicad_sch (KiCad schematic)
At the start: 4 parts, among them J5 XLR3, J7 XLR3, SW3 SW_DIP_x02

Commit message: finalisation PCB-salle de Répétition
Parts:
- U8: footprint (none) -> Relais_Sig:IM43GR
- renumbered J5 to J7, J7 to J8
Other:
- moved on the sheet: SW3, U8

Commit message: finalisation v2 PCB repetition
Connections:
- net GND1 is gone; now on net GND: SW3.1
- net GND: no longer J8.1, SW3.4
- net GND2 renamed GND_entree
- new net GND_sortie: J8.1, SW3.4
Changed lines of the file:
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@@
 	(paper "A4")
 	(rectangle
-		(start 177.038 38.354)
+		(start 171.45 38.354)
 		(end 213.36 100.838)
 		(stroke
@@
 		)
 	)
-	(junction
-		(at 110.49 41.91)
-		(diameter 0)
-		(color 0 0 0 0)
-	)
 	(wire
 		(pts
-			(xy 110.49 39.37) (xy 109.22 39.37)
+			(xy 119.38 39.37) (xy 109.22 39.37)
 		)
 		(stroke
@@
 	(wire
 		(pts
-			(xy 110.49 39.37) (xy 110.49 41.91)
+			(xy 82.55 41.91) (xy 93.98 41.91)
 		)
 		(stroke
@@
 		)
 	)
-	(wire
-		(pts
-			(xy 87.63 41.91) (xy 93.98 41.91)
-		)
-		(stroke
-			(width 0)
-			(type default)
-		)
-	)
-	(wire
-		(pts
-			(xy 110.49 41.91) (xy 109.22 41.91)
-		)
-		(stroke
-			(width 0)
-			(type default)
-		)
-	)
 	(label "OUT+"
 		(at 201.93 67.31 0)
@@
 		)
 	)
-	(label "GND2"
-		(at 87.63 41.91 0)
-		(effects
-			(font
-				(size 1.27 1.27)
-			)
-			(justify left bottom)
-		)
-	)
 	(label "IN+"
 		(at 153.67 68.58 0)
@@
 		)
 	)
-	(label "GND2"
+	(label "GND_entree"
 		(at 138.43 68.58 180)
 		(effects
@@
 			)
 			(justify right bottom)
+		)
+	)
+	(label "GND_sortie"
+		(at 119.38 39.37 180)
+		(effects
+			(font
+				(size 1.27 1.27)
+			)
+			(justify right bottom)
+		)
+	)
+	(label "GND_entree"
+		(at 82.55 41.91 0)
+		(effects
+			(font
+				(size 1.27 1.27)
+			)
+			(justify left bottom)
 		)
 	)
@@
 			)
 			(justify left bottom)
+		)
+	)
+	(label "GND_sortie"
+		(at 186.69 67.31 180)
+		(effects
+			(font
+				(size 1.27 1.27)
+			)
+			(justify right bottom)
 		)
 	)
@@
 			)
 			(justify left)
-		)
-	)
-	(hierarchical_label "GND1"
-		(shape input)
-		(at 93.98 39.37 180)
-		(effects
-			(font
-				(size 1.27 1.27)
-			)
-			(justify right)
 		)
 	)
@@
 	)
 	(symbol
-		(lib_id "power:GND")
-		(at 186.69 67.31 0)
-		(unit 1)
-		(exclude_from_sim no)
-		(in_bom yes)
-		(on_board yes)
-		(dnp no)
-		(fields_autoplaced yes)
-		(property "Reference" "#PWR063"
-			(at 186.69 73.66 0)
-			(effects
-				(font
-					(size 1.27 1.27)
-				)
-				(hide yes)
-			)
-		)
-		(property "Value" "GND"
-			(at 186.69 72.136 0)
-			(effects
-				(font
-					(size 1.27 1.27)
-				)
-			)
-		)
-		(property "Footprint" ""
-			(at 186.69 67.31 0)
-			(effects
-				(font
-					(size 1.27 1.27)
-				)
-				(hide yes)
-			)
-		)
-		(property "Datasheet" ""
-			(at 186.69 67.31 0)
-			(effects
-				(font
-					(size 1.27 1.27)
-				)
-				(hide yes)
-			)
-		)
-		(property "Description" "Power symbol creates a global label with name \"GND\" , ground"
-			(at 186.69 67.31 0)
-			(effects
-				(font
-					(size 1.27 1.27)
-				)
-				(hide yes)
-			)
-		)
-		(pin "1"
-		)
-		(instances
-			(project "PCB_Repetition"
-				(path "/256ff558-4730-4071-bd27-80924a9e3a69/7143666d-a23b-4ee4-b5d7-a29986b50a19"
-					(reference "#PWR067")
-					(unit 1)
-				)
-				(path "/256ff558-4730-4071-bd27-80924a9e3a69/8626c1d5-5981-47d9-9975-892e686a3aac"
-					(reference "#PWR065")
-					(unit 1)
-				)
-				(path "/256ff558-4730-4071-bd27-80924a9e3a69/8c759eb1-d9e1-4a15-beba-1b103a9d9af9"
-					(reference "#PWR063")
-					(unit 1)
-				)
-				(path "/256ff558-4730-4071-bd27-80924a9e3a69/9d3d58f4-fdb6-4bae-b68b-9954abd46f82"
-					(reference "#PWR073")
-					(unit 1)
-				)
-				(path "/256ff558-4730-4071-bd27-80924a9e3a69/ae810da9-ce25-4571-894f-4d416f910cb9"
-					(reference "#PWR071")
-					(unit 1)
-				)
-				(path "/256ff558-4730-4071-bd27-80924a9e3a69/b54643fa-e62f-4566-ace2-5f15832f1805"
-					(reference "#PWR069")
-					(unit 1)
-				)
-			)
-		)
-	)
-	(symbol
 		(lib_id "Connector_Audio:XLR3")
 		(at 146.05 68.58 0)
@@
 	(symbol
 		(lib_id "power:GND")
-		(at 110.49 41.91 0)
+		(at 109.22 41.91 0)
 		(unit 1)
 		(exclude_from_sim no)
@@
 		(fields_autoplaced yes)
 		(property "Reference" "#PWR062"
-			(at 110.49 48.26 0)
+			(at 109.22 48.26 0)
 			(effects
 				(font
@@
 		)
 		(property "Value" "GND"
-			(at 110.49 46.736 0)
-			(effects
-				(font
-					(size 1.27 1.27)
-				)
+			(at 109.22 46.99 0)
+			(effects
+				(font
+					(size 1.27 1.27)
+				)
+				(hide yes)
 			)
 		)
 		(property "Footprint" ""
-			(at 110.49 41.91 0)
+			(at 109.22 41.91 0)
 			(effects
 				(font
@@
 		)
 		(property "Datasheet" ""
-			(at 110.49 41.91 0)
+			(at 109.22 41.91 0)
 			(effects
 				(font
@@
 		)
 		(property "Description" "Power symbol creates a global label with name \"GND\" , ground"
-			(at 110.49 41.91 0)
+			(at 109.22 41.91 0)
 			(effects
 				(font
@@
 					(unit 1)
 				)
+			)
+		)
+	)
+	(symbol
+		(lib_id "power:GND")
+		(at 93.98 39.37 180)
+		(unit 1)
+		(exclude_from_sim no)
+		(in_bom yes)
+		(on_board yes)
+		(dnp no)
+		(fields_autoplaced yes)
+		(property "Reference" "#PWR024"
+			(at 93.98 33.02 0)
+			(effects
+				(font
+					(size 1.27 1.27)
+				)
+				(hide yes)
+			)
+		)
+		(property "Value" "GND"
+			(at 93.98 34.29 0)
+			(effects
+				(font
+					(size 1.27 1.27)
+				)
+				(hide yes)
+			)
+		)
+		(property "Footprint" ""
+			(at 93.98 39.37 0)
+			(effects
+				(font
+					(size 1.27 1.27)
+				)
+				(hide yes)
+			)
+		)
+		(property "Datasheet" ""
+			(at 93.98 39.37 0)
+			(effects
+				(font
+					(size 1.27 1.27)
+				)
+				(hide yes)
+			)
+		)
+		(property "Description" "Power symbol creates a global label with name \"GND\" , ground"
+			(at 93.98 39.37 0)
+			(effects
+				(font
+					(size 1.27 1.27)
+				)
+				(hide yes)
+			)
+		)
+		(pin "1"
+		)
+		(instances
+			(project "PCB_Repetition"
+				(path "/256ff558-4730-4071-bd27-80924a9e3a69/7143666d-a23b-4ee4-b5d7-a29986b50a19"
+					(reference "#PWR028")
+					(unit 1)
+				)
+				(path "/256ff558-4730-4071-bd27-80924a9e3a69/8626c1d5-5981-47d9-9975-892e686a3aac"
+					(reference "#PWR025")
+					(unit 1)
+				)
+				(path "/256ff558-4730-4071-bd27-80924a9e3a69/8c759eb1-d9e1-4a15-beba-1b103a9d9af9"
+					(reference "#PWR024")
+					(unit 1)
+				)
+				(path "/256ff558-4730-4071-bd27-80924a9e3a69/9d3d58f4-fdb6-4bae-b68b-9954abd46f82"
+					(reference "#PWR075")
+					(unit 1)
+				)
+				(path "/256ff558-4730-4071-bd27-80924a9e3a69/ae810da9-ce25-4571-894f-4d416f910cb9"
+					(reference "#PWR074")
+					(unit 1)
+				)
+				(path "/256ff558-4730-4071-bd27-80924a9e3a69/b54643fa-e62f-4566-ace2-5f15832f1805"
+					(reference "#PWR031")
+					(unit 1)
+				)
